Commit message: Add files via upload
Minor updates - May 2024

File: description/camera.xacro (robot description, xacro)
@@ -2,8 +2,8 @@
 <robot xmlns:xacro="http://www.ros.org/wiki/xacro" >
     <!-- ********************** CAMERA CONSTANTS *********************************  -->
-    <xacro:property name="camera_height" value="0.075" />
+    <xacro:property name="camera_height" value="0.08" />
     <xacro:property name="camera_width" value="0.02" />
     <xacro:property name="camera_thick" value="0.01" />
-    <xacro:property name="camera_x" value="0.04" />
+    <xacro:property name="camera_x" value="0.03" />
     <xacro:property name="camera_y" value="0.025" />
     <xacro:property name="camera_z" value="0.05" />
@@ -22,9 +22,4 @@
             <material name="Green" />
         </visual>
-        <inertial>
-            <origin xyz="${camera_x} ${camera_y} ${camera_z}" rpy="0 0 0" />
-            <mass value="0.1" />
-            <inertia ixx="0.0" ixy="0.0" ixz="0.0" iyy="0.0" iyz="0.0" izz="0.0" />
-        </inertial>
         <collision>
             <origin xyz="${camera_x} ${camera_y} ${camera_z}" rpy="0 0 0"/>
@@ -33,13 +28,18 @@
             </geometry>
         </collision>
+        <inertial>
+            <origin xyz="${camera_x} ${camera_y} ${camera_z}" rpy="0 0 0" />
+            <mass value="${mass}" />
+            <inertia ixx="${inertia}" ixy="0.0" ixz="0.0" iyy="${inertia}" iyz="0.0" izz="${inertia}" />
+        </inertial>
     </link>
     <joint name="camera_optical_joint" type="fixed">
         <parent link="camera_link"/>
         <child link="camera_link_optical"/>
-        <origin xyz="0 0 0" rpy="${-pi/2} 0 ${-pi/2}"/>
+        <origin xyz="${camera_x} ${camera_y} ${camera_z}" rpy="0 0 0"/>
     </joint>
     <link name="camera_link_optical"></link>
     <!-- ********************** Gazebo Characteristics *********************************  -->
-    <gazebo reference="camera_link">
+    <gazebo reference="camera_link_optical">
         <material>Gazebo/Green</material>
         <sensor name="camera" type="camera">
@@ -60,5 +60,16 @@
             </camera>
             <plugin name="camera_controller" filename="libgazebo_ros_camera.so">
-                <frame_name>camera_link_optical</frame_name>
+                <alwaysOn>true</alwaysOn>
+                <updateRate>0.0</updateRate>
+                <cameraName>bartrover/camera1</cameraName>
+                <frameName>camera_link_optical</frameName>
+                <imageTopicName>image_raw</imageTopicName>
+                <cameraInfoTopicName>camera_info</cameraInfoTopicName>
+                <hackBaseline>0.07</hackBaseline>
+                <distortionK1>0.0</distortionK1>
+                <distortionK2>0.0</distortionK2>
+                <distortionK3>0.0</distortionK3>
+                <distortionT1>0.0</distortionT1>
+                <distortionT2>0.0</distortionT2>
             </plugin>
         </sensor>

File: description/gazebo_control.xacro (robot description, xacro)
@@ -3,6 +3,6 @@
     <gazebo>
         <plugin name="diff_drive" filename="libgazebo_ros_diff_drive.so">
-            <!-- Number of wheel pairs
-            <num_wheel_pairs>3</num_wheel_pairs> -->
+            <!-- Number of wheel pairs -->
+            <num_wheel_pairs>3</num_wheel_pairs>
             <!-- Wheel Information -->
             <left_joint>rear_left_wheel_joint</left_joint>

File: description/lidar.xacro (robot description, xacro)
@@ -1,13 +1,17 @@
 <?xml version="1.0"?>
 <robot xmlns:xacro="http://www.ros.org/wiki/xacro" >
+    <!-- ********************** LIDAR CONSTANTS *********************************  -->
+    <xacro:property name="lidar_x" value="-0.01" />
+    <xacro:property name="lidar_y" value="-0.012" />
+    <xacro:property name="lidar_z" value="0.045" />
     <!-- ********************** Physical Characteristics *********************************  -->
     <joint name="laser_joint" type="fixed">
         <parent link="body_link"/>
         <child link="laser_frame"/>
-        <origin xyz="0.08 -0.01 0.08" rpy="0 0 0"/>
+        <origin xyz="${lidar_x} ${lidar_y} ${lidar_z}" rpy="0 0 0"/>
     </joint>
     <link name="laser_frame">
         <visual>
-            <origin xyz="-0.01 -0.01 0" rpy="0 0 0" />
+            <origin xyz="${lidar_x} ${lidar_y} ${lidar_z}" rpy="0 0 0" />
             <geometry>
                 <cylinder radius="0.035" length="0.05"/>
@@ -16,5 +20,5 @@
         </visual>
         <collision>
-            <origin xyz="-0.01 -0.01 0" rpy="0 0 0"/>
+            <origin xyz="${lidar_x} ${lidar_y} ${lidar_z}" rpy="0 0 0"/>
             <geometry>
                 <cylinder radius="0.035" length="0.05"/>
@@ -22,5 +26,5 @@
         </collision>
         <xacro:inertial_cylinder mass="0.1" length="0.05" radius="0.035">
-            <origin xyz="-0.01 -0.01 0" rpy="0 0 0" />
+            <origin xyz="${lidar_x} ${lidar_y} ${lidar_z}" rpy="0 0 0" />
         </xacro:inertial_cylinder>
     </link>

File: description/ros2_control.xacro (robot description, xacro)
@@ -7,4 +7,8 @@
                 <param name="rear_left_wheel_name">rear_left_wheel_joint</param>
                 <param name="rear_right_wheel_name">rear_right_wheel_joint</param>
+                <param name="middle_left_wheel_name">middle_left_wheel_joint</param>
+                <param name="middle_right_wheel_name">middle_right_wheel_joint</param>
+                <param name="front_left_wheel_name">front_left_wheel_joint</param>
+                <param name="front_right_wheel_name">front_right_wheel_joint</param>
                 <param name="loop_rate">30</param>
                 <param name="device">/dev/ttyUSB0</param>
@@ -13,4 +17,5 @@
                 <param name="enc_counts_per_rev">3436</param>
             </hardware>
+            <!-- ********************** REAR ********************************* -->
             <joint name="rear_left_wheel_joint">
                 <command_interface name="velocity">
@@ -29,4 +34,38 @@
                 <state_interface name="velocity"/>
             </joint>
+            <!-- ********************** MIDDLE ********************************* -->
+            <joint name="middle_left_wheel_joint">
+                <command_interface name="velocity">
+                    <param name="min">-10</param>
+                    <param name="max">10</param>
+                </command_interface>
+                <state_interface name="position"/>
+                <state_interface name="velocity"/>
+            </joint>
+            <joint name="middle_right_wheel_joint">
+                <command_interface name="velocity">
+                    <param name="min">-10</param>
+                    <param name="max">10</param>
+                </command_interface>
+                <state_interface name="position"/>
+                <state_interface name="velocity"/>
+            </joint>
+            <!-- ********************** FORWARD ********************************* -->
+            <joint name="front_left_wheel_joint">
+                <command_interface name="velocity">
+                    <param name="min">-10</param>
+                    <param name="max">10</param>
+                </command_interface>
+                <state_interface name="position"/>
+                <state_interface name="velocity"/>
+            </joint>
+            <joint name="front_right_wheel_joint">
+                <command_interface name="velocity">
+                    <param name="min">-10</param>
+                    <param name="max">10</param>
+                </command_interface>
+                <state_interface name="position"/>
+                <state_interface name="velocity"/>
+            </joint>
         </ros2_control>
     </xacro:unless>
@@ -36,4 +75,5 @@
                 <plugin>gazebo_ros2_control/GazeboSystem</plugin>
             </hardware>
+            <!-- ********************** REAR ********************************* -->
             <joint name="rear_left_wheel_joint">
                 <command_interface name="velocity">
@@ -52,4 +92,38 @@
                 <state_interface name="velocity"/>
             </joint>
+            <!-- ********************** MIDDLE ********************************* -->
+            <joint name="middle_left_wheel_joint">
+                <command_interface name="velocity">
+                    <param name="min">-10</param>
+                    <param name="max">10</param>
+                </command_interface>
+                <state_interface name="position"/>
+                <state_interface name="velocity"/>
+            </joint>
+            <joint name="middle_right_wheel_joint">
+                <command_interface name="velocity">
+                    <param name="min">-10</param>
+                    <param name="max">10</param>
+                </command_interface>
+                <state_interface name="position"/>
+                <state_interface name="velocity"/>
+            </joint>
+            <!-- ********************** FORWARD ********************************* -->
+            <joint name="front_left_wheel_joint">
+                <command_interface name="velocity">
+                    <param name="min">-10</param>
+                    <param name="max">10</param>
+                </command_interface>
+                <state_interface name="position"/>
+                <state_interface name="velocity"/>
+            </joint>
+            <joint name="front_right_wheel_joint">
+                <command_interface name="velocity">
+                    <param name="min">-10</param>
+                    <param name="max">10</param>
+                </command_interface>
+                <state_interface name="position"/>
+                <state_interface name="velocity"/>
+            </joint>
         </ros2_control>
     </xacro:if>
