Commit message: Add files via upload

File: description/bartrover.xacro (robot description, xacro)
@@ -7,5 +7,4 @@
     <xacro:include filename="lidar.xacro" />
     <xacro:include filename="camera.xacro" />
-    <!-- <xacro:include filename="depth_camera.xacro" /> -->
     <xacro:if value="$(arg use_ros2_control)">
         <xacro:include filename="ros2_control.xacro" />

File: description/bartrover_core.xacro (robot description, xacro)
@@ -24,5 +24,5 @@
 			<origin xyz="0 0 0.03" rpy="0 0 0" />
             <geometry>
-                <box size="0.28 ${wheel_separation} 0.08"/>
+                <box size="${body_length} ${wheel_separation} ${body_height}"/>
             </geometry>
 			<material name="White" />
@@ -31,13 +31,11 @@
 			<origin xyz="0 0 0.03" rpy="0 0 0" />
             <geometry>
-                <box size="0.28 ${wheel_separation} 0.08"/>
+                <box size="${body_length} ${wheel_separation} ${body_height}"/>
             </geometry>
 		</collision>
-        <inertial>
-            <origin xyz="0 0 0.03" rpy="0 0 0" />
-            <mass value="${mass}" />
-            <inertia ixx="${inertia}" ixy="0.0" ixz="0.0" iyy="${inertia}" iyz="0.0" izz="${inertia}" />
-        </inertial>
-	</link>
+        <xacro:inertial_box mass="${body_mass}" x="${body_length}" y="${wheel_separation}" z="${body_height}">
+            <origin xyz="0 0 0.03" rpy="0 0 0"/>
+        </xacro:inertial_box>
+    </link>
     <gazebo reference="body_link">
         <material>Gazebo/White</material>
@@ -50,4 +48,6 @@
         <origin xyz="-0.104 ${wheel_separation/2 + wheel_width/2} 0" rpy="0 0 0"/>
         <axis xyz="0 1 0"/>
+        <limit effort="${limit_effort}" velocity="${limit_velocity}"/>
+        <dynamics damping="${dynamic_damping}" friction="${spinning_friction}"/>
     </joint>
     <link name="rear_left_wheel">
@@ -105,4 +105,6 @@
 		<origin xyz="-0.104 ${-1 * (wheel_separation/2 + wheel_width/2)} 0" rpy="0 0 0"/>
         <axis xyz="0 1 0"/>
+        <limit effort="${limit_effort}" velocity="${limit_velocity}"/>
+        <dynamics damping="${dynamic_damping}" friction="${spinning_friction}"/>
     </joint>
     <link name="rear_right_wheel">
@@ -161,4 +163,6 @@
 		<origin xyz="0 ${wheel_separation/2 + wheel_width/2} 0" rpy="0 0 0" />
         <axis xyz="0 1 0"/>
+        <limit effort="${limit_effort}" velocity="${limit_velocity}"/>
+        <dynamics damping="${dynamic_damping}" friction="${spinning_friction}"/>
     </joint>
     <link name="middle_left_wheel">
@@ -216,4 +220,6 @@
 		<origin xyz="0 ${-1 * (wheel_separation/2 + wheel_width/2)} 0" rpy="0 0 0" />
         <axis xyz="0 1 0"/>
+        <limit effort="${limit_effort}" velocity="${limit_velocity}"/>
+        <dynamics damping="${dynamic_damping}" friction="${spinning_friction}"/>
     </joint>
     <link name="middle_right_wheel">
@@ -272,4 +278,6 @@
 		<origin xyz="0.104 ${wheel_separation/2 + wheel_width/2} 0" rpy="0 0 0" />
         <axis xyz="0 1 0"/>
+        <limit effort="${limit_effort}" velocity="${limit_velocity}"/>
+        <dynamics damping="${dynamic_damping}" friction="${spinning_friction}"/>
     </joint>
     <link name="front_left_wheel">
@@ -327,4 +335,6 @@
 		<origin xyz="0.104 ${-1 * (wheel_separation/2 + wheel_width/2)} 0" rpy="0 0 0" />
         <axis xyz="0 1 0"/>
+        <limit effort="${limit_effort}" velocity="${limit_velocity}"/>
+        <dynamics damping="${dynamic_damping}" friction="${spinning_friction}"/>
     </joint>
     <link name="front_right_wheel">

File: description/camera.xacro (robot description, xacro)
@@ -2,19 +2,19 @@
 <robot xmlns:xacro="http://www.ros.org/wiki/xacro" >
     <!-- ********************** CAMERA CONSTANTS *********************************  -->
-    <xacro:property name="camera_height" value="0.08" />
+    <xacro:property name="camera_height" value="0.04" />
     <xacro:property name="camera_width" value="0.02" />
     <xacro:property name="camera_thick" value="0.01" />
-    <xacro:property name="camera_x" value="0.03" />
-    <xacro:property name="camera_y" value="0.025" />
-    <xacro:property name="camera_z" value="0.05" />
+    <xacro:property name="camera_x" value="0.12" />
+    <xacro:property name="camera_y" value="0.02" />
+    <xacro:property name="camera_z" value="0.064" />
     <!-- ********************** Physical Characteristics *********************************  -->
     <joint name="camera_joint" type="fixed">
         <parent link="body_link"/>
-        <child link="camera_link"/>
+        <child link="camera"/>
         <origin xyz="${camera_x} ${camera_y} ${camera_z}" rpy="0 0 0"/>
     </joint>
-    <link name="camera_link">
+    <link name="camera">
         <visual>
-            <origin xyz="${camera_x} ${camera_y} ${camera_z}" rpy="0 0 0" />
+            <origin xyz="${camera_x - .1} ${camera_y} ${camera_z -.072}" rpy="0 0 0" />
             <geometry>
                 <box size="${camera_thick} ${camera_width} ${camera_height}" />
@@ -22,24 +22,7 @@
             <material name="Green" />
         </visual>
-        <collision>
-            <origin xyz="${camera_x} ${camera_y} ${camera_z}" rpy="0 0 0"/>
-            <geometry>
-                <box size="${camera_thick} ${camera_width} ${camera_height}"/>
-            </geometry>
-        </collision>
-        <inertial>
-            <origin xyz="${camera_x} ${camera_y} ${camera_z}" rpy="0 0 0" />
-            <mass value="${mass}" />
-            <inertia ixx="${inertia}" ixy="0.0" ixz="0.0" iyy="${inertia}" iyz="0.0" izz="${inertia}" />
-        </inertial>
     </link>
-    <joint name="camera_optical_joint" type="fixed">
-        <parent link="camera_link"/>
-        <child link="camera_link_optical"/>
-        <origin xyz="${camera_x} ${camera_y} ${camera_z}" rpy="0 0 0"/>
-    </joint>
-    <link name="camera_link_optical"></link>
     <!-- ********************** Gazebo Characteristics *********************************  -->
-    <gazebo reference="camera_link_optical">
+    <gazebo reference="camera">
         <material>Gazebo/Green</material>
         <sensor name="camera" type="camera">
@@ -47,5 +30,8 @@
             <visualize>true</visualize>
             <update_rate>10</update_rate>
+            <topic>camera/image_raw</topic>
+            <gz_frame_id>camera_rgb_frame</gz_frame_id>
             <camera>
+                <camera_info_topic>camera/camera_info</camera_info_topic>
                 <horizontal_fov>1.089</horizontal_fov>
                 <image>
@@ -58,13 +44,18 @@
                     <far>8.0</far>
                 </clip>
+                <noise>
+                    <type>gaussian</type>
+                    <mean>0.0</mean>
+                    <stddev>0.007</stddev>
+                </noise>
             </camera>
+<!--
             <plugin name="camera_controller" filename="libgazebo_ros_camera.so">
-                <frameName>camera_link_optical</frameName>
-            <!--
                 <alwaysOn>true</alwaysOn>
                 <updateRate>0.0</updateRate>
-                <cameraName>bartrover/camera1</cameraName>
+                <cameraName>camera</cameraName>
                 <imageTopicName>image_raw</imageTopicName>
                 <cameraInfoTopicName>camera_info</cameraInfoTopicName>
+                <frameName>camera</frameName>
                 <hackBaseline>0.07</hackBaseline>
                 <distortionK1>0.0</distortionK1>
@@ -73,6 +64,6 @@
                 <distortionT1>0.0</distortionT1>
                 <distortionT2>0.0</distortionT2>
-            -->
             </plugin>
+-->
         </sensor>
     </gazebo>

File: description/constants_macros.xacro (robot description, xacro)
@@ -3,13 +3,17 @@
     <!-- Specify Some Useful Robot Constants -->
     <!-- ********************** ROBOT CONSTANTS *********************************  -->
+    <xacro:property name="PI" value="3.1415926"/>
     <xacro:property name="clearance" value="0.035" />
+    <xacro:property name="body_length" value="0.28"/>
+    <xacro:property name="body_height" value="0.08"/>
+    <xacro:property name="wheel_separation" value="0.15"/>
     <xacro:property name="wheel_radius" value="0.035"/>
-    <xacro:property name="wheel_separation" value="0.15"/>
     <xacro:property name="wheel_width" value="0.035"/>
-    <xacro:property name="mass" value="0.1"/>
-    <xacro:property name="wheel_mass" value="0.2"/>
+    <xacro:property name="steel_density" value="7850"/> <!--Steel-->
+    <xacro:property name="body_density" value="${steel_density/3}"/>
+    <xacro:property name="wheel_density" value="900"/> <!--Rubber-->
+    <xacro:property name="body_mass" value="${body_density * body_length * body_height * wheel_separation}"/>
+    <xacro:property name="wheel_mass" value="${wheel_density * PI * wheel_radius * wheel_radius * wheel_width}"/>
     <xacro:property name="marker_mass" value="0.0"/>
-    <xacro:property name="inertia" value="0.3"/>
-    <xacro:property name="PI" value="3.1415926"/>
     <xacro:property name="wheel_ixx" value="${wheel_mass*(3*wheel_radius*wheel_radius+wheel_width*wheel_width)/12}" />
     <xacro:property name="wheel_ixy" value="0.0" />
@@ -18,4 +22,7 @@
     <xacro:property name="wheel_iyz" value="0.0" />
     <xacro:property name="wheel_izz" value="${wheel_mass*wheel_radius*wheel_radius/2}" />
+    <xacro:property name="dynamic_damping" value="0.1" />
+    <xacro:property name="limit_effort" value="100" />
+    <xacro:property name="limit_velocity" value="10" />
     <!-- ********************** GAZEBO CONSTANTS *********************************  -->
     <xacro:property name="lateral_friction" value="1.0" />

File: description/gazebo_control.xacro (robot description, xacro)
@@ -2,5 +2,5 @@
 <robot xmlns:xacro="http://www.ros.org/wiki/xacro">
     <gazebo>
-        <plugin name="diff_drive" filename="libgazebo_ros_diff_drive.so">
+        <plugin name="gz::sim::systems::DiffDrive" filename="gz-sim-diff-drive-system">
             <!-- Number of wheel pairs -->
             <num_wheel_pairs>3</num_wheel_pairs>
@@ -9,24 +9,38 @@
             <right_joint>rear_right_wheel_joint</right_joint>
             <wheel_separation>0.15</wheel_separation>
-            <wheel_diameter>0.07</wheel_diameter>
+            <wheel_radius>0.035</wheel_radius>
             <left_joint>middle_left_wheel_joint</left_joint>
             <right_joint>middle_right_wheel_joint</right_joint>
             <wheel_separation>0.15</wheel_separation>
-            <wheel_diameter>0.07</wheel_diameter>
+            <wheel_radius>0.035</wheel_radius>
             <left_joint>front_left_wheel_joint</left_joint>
             <right_joint>front_right_wheel_joint</right_joint>
             <wheel_separation>0.15</wheel_separation>
-            <wheel_diameter>0.07</wheel_diameter>
-            <update_rate>30</update_rate>
+            <wheel_radius>0.035</wheel_radius>
             <!-- Limits -->
-            <max_wheel_torque>200</max_wheel_torque>
-            <max_wheel_acceleration>10.0</max_wheel_acceleration>
+            <max_linear_acceleration>0.33</max_linear_acceleration>
+            <max_wheel_torque>20</max_wheel_torque>
+            <!-- Input -->
+            <topic>cmd_vel</topic>
             <!-- Output -->
-            <odometry_frame>odom</odometry_frame>
-            <robot_base_frame>base_link</robot_base_frame>
+            <frame_id>odom</frame_id>
+            <child_frame_id>body_link</child_frame_id>
+            <odom_topic>odom</odom_topic>
+            <odom_publish_frequency>30</odom_publish_frequency>
+            <tf_topic>/tf</tf_topic>
             <publish_odom>true</publish_odom>
             <publish_odom_tf>true</publish_odom_tf>
             <publish_wheel_tf>true</publish_wheel_tf>
         </plugin>
+        <plugin filename="gz-sim-joint-state-publisher-system" name="gz::sim::systems::JointStatePublisher">
+            <topic>joint_states</topic>
+            <update_rate>50</update_rate>
+            <joint_name>rear_left_wheel_joint</joint_name>
+            <joint_name>rear_right_wheel_joint</joint_name>
+            <joint_name>middle_left_wheel_joint</joint_name>
+            <joint_name>middle_right_wheel_joint</joint_name>
+            <joint_name>front_left_wheel_joint</joint_name>
+            <joint_name>front_right_wheel_joint</joint_name>
+        </plugin>
     </gazebo>
 </robot>

File: description/lidar.xacro (robot description, xacro)
@@ -2,39 +2,44 @@
 <robot xmlns:xacro="http://www.ros.org/wiki/xacro" >
     <!-- ********************** LIDAR CONSTANTS *********************************  -->
-    <xacro:property name="lidar_x" value="-0.01" />
-    <xacro:property name="lidar_y" value="-0.012" />
-    <xacro:property name="lidar_z" value="0.045" />
+    <xacro:property name="lidar_x" value="0.04" />
+    <xacro:property name="lidar_y" value="0.0" />
+    <xacro:property name="lidar_z" value="0.04" />
+    <xacro:property name="lidar_rad" value="0.035" />
+    <xacro:property name="lidar_ht" value="0.02" />
     <!-- ********************** Physical Characteristics *********************************  -->
-    <joint name="laser_joint" type="fixed">
+    <joint name="lidar_joint" type="fixed">
         <parent link="body_link"/>
-        <child link="laser_frame"/>
-        <origin xyz="${lidar_x} ${lidar_y} ${lidar_z}" rpy="0 0 0"/>
+        <child link="lidar"/>
+        <origin xyz="${lidar_x} ${lidar_y} ${lidar_z +.05}" rpy="0 0 0"/>
     </joint>
-    <link name="laser_frame">
+    <link name="lidar">
         <visual>
-            <origin xyz="${lidar_x} ${lidar_y} ${lidar_z}" rpy="0 0 0" />
+            <origin xyz="${lidar_x} ${lidar_y} ${lidar_z -.05}" rpy="0 0 0" />
             <geometry>
-                <cylinder radius="0.035" length="0.05"/>
+                <cylinder radius="${lidar_rad}" length="${lidar_ht}"/>
             </geometry>
             <material name="Blue" />
         </visual>
         <collision>
-            <origin xyz="${lidar_x} ${lidar_y} ${lidar_z}" rpy="0 0 0"/>
+            <origin xyz="${lidar_x} ${lidar_y} ${lidar_z - .05}" rpy="0 0 0"/>
             <geometry>
-                <cylinder radius="0.035" length="0.05"/>
+                <cylinder radius="${lidar_rad}" length="${lidar_ht}"/>
             </geometry>
         </collision>
-        <xacro:inertial_cylinder mass="0.1" length="0.05" radius="0.035">
-            <origin xyz="${lidar_x} ${lidar_y} ${lidar_z}" rpy="0 0 0" />
+        <xacro:inertial_cylinder mass="0.1" length="${lidar_ht}" radius="${lidar_rad}">
+            <origin xyz="${lidar_x} ${lidar_y} ${lidar_z - .05}" rpy="0 0 0" />
         </xacro:inertial_cylinder>
     </link>
     <!-- ********************** Gazebo Characteristics *********************************  -->
-    <gazebo reference="laser_frame">
+    <gazebo reference="lidar">
         <material>Gazebo/Blue</material>
-        <sensor name="laser" type="ray">
+        <sensor name="lidar" type="gpu_lidar">
             <pose> 0 0 0 0 0 0 </pose>
-            <visualize>false</visualize>
+            <always_on>true</always_on>
+            <visualize>true</visualize>
             <update_rate>10</update_rate>
-            <ray>
+            <topic>scan</topic>
+            <gz_frame_id>base_scan</gz_frame_id>
+            <lidar>
                 <scan>
                     <horizontal>
@@ -47,13 +52,22 @@
                     <min>0.3</min>
                     <max>12</max>
+                    <resolution>0.01</resolution>
                 </range>
-            </ray>
+                <noise>
+                    <type>gaussian</type>
+                    <mean>0.0</mean>
+                    <stddev>0.001</stddev>
+                </noise>
+            </lidar>
+ <!--
             <plugin name="laser_controller" filename="libgazebo_ros_ray_sensor.so">
                 <ros>
-                    <argument>~/out:=scan</argument>
+                    <namespace>/</namespace>
+                    <remapping>~/out:=scan</remapping>
                 </ros>
                 <output_type>sensor_msgs/LaserScan</output_type>
-                <frame_name>laser_frame</frame_name>
+                <frame_name>lidar</frame_name>
             </plugin>
+-->
         </sensor>
     </gazebo>

File: description/ros2_control.xacro (robot description, xacro)
@@ -4,5 +4,6 @@
         <ros2_control name="RealRobot" type="system">
             <hardware>
-                <plugin>diffdrive_arduino/DiffDriveArduinoHardware</plugin>
+                <!-- <plugin>diffdrive_arduino/DiffDriveArduinoHardware</plugin>-->
+                <plugin>diffdrive_arduino/DiffDriveArduino</plugin>
                 <param name="left_wheel_name">rear_left_wheel_joint</param>
                 <param name="right_wheel_name">rear_right_wheel_joint</param>
@@ -10,5 +11,6 @@
                 <param name="device">/dev/ttyUSB0</param>
                 <param name="baud_rate">57600</param>
-                <param name="timeout_ms">1000</param>
+                <!-- <param name="timeout_ms">1000</param>-->
+                <param name="timeout">1000</param>
                 <param name="enc_counts_per_rev">3436</param>
             </hardware>
@@ -73,5 +75,5 @@
         <ros2_control name="GazeboSystem" type="system">
             <hardware>
-                <plugin>gazebo_ros2_control/GazeboSystem</plugin>
+                <plugin>gz_ros2_control/GazeboSimSystem</plugin>
             </hardware>
             <!-- ********************** REAR ********************************* -->
@@ -129,5 +131,5 @@
     </xacro:if>
     <gazebo>
-        <plugin name="gazebo_ros2_control" filename="libgazebo_ros2_control.so">
+        <plugin name="gz_ros2_control::GazeboSimROS2ControlPlugin" filename="libgz_ros2_control-system.so">
             <parameters>$(find bartrover)/config/my_controllers.yaml</parameters>
             <parameters>$(find bartrover)/config/gaz_ros2_ctl_use_sim.yaml</parameters>
